File: tmc2208-breakout.kicad_pcb (KiCad board)
At the start: 2 copper layers, 31 x 36 mm, 41 parts, among them J1 Conn_01x05, J2 Conn_01x05, J3 Conn_01x04, J4 Conn_01x02, U1 TMC2208-LA

Commit message: changed some minor things like connector and finalized bom for v1.0
Parts:
- removed J2: Conn_01x05, Connector_PinHeader_2.54mm:PinHeader_1x05_P2.54mm_Vertical
- C7: footprint Capacitor_SMD:CP_Elec_5x5.4 -> Capacitor_SMD:CP_Elec_6.3x5.4
- J1: value Conn_01x05 -> Conn_01x11; footprint Connector_PinHeader_2.54mm:PinHeader_1x05_P2.54mm_Vertical -> Connector_PinHeader_2.54mm:PinHeader_1x11_P2.54mm_Vertical
- R8: value R -> 0
- TP1: renamed from EN#; value TestPoint -> EN#
- TP2: renamed from DIR; value TestPoint -> DIR
- TP3: renamed from MS1; value TestPoint -> MS1
- TP4: renamed from MS2; value TestPoint -> MS2
- TP5: renamed from STEP; value TestPoint -> STEP
- TP6: renamed from DIAG; value TestPoint -> DIAG
- TP7: renamed from INDX; value TestPoint -> INDX
- TP8: renamed from PDN; value TestPoint -> PDN
- moved J1 2.42 mm to (144.0, 41.5)
- moved C7 2.06 mm to (157.5, 46.0)
Connections:
- J1 pad 2: /STEP -> /VREF
- J1 pad 3: /EN# -> /STEP
- J1 pad 4: /MS1 -> /EN#
- J1 pad 5: /MS2 -> /MS1
Routing:
- net /VREF: track 4.79 -> 31.9 mm, vias 0 -> 1
- net /VS: track 57.9 -> 61.3 mm
- net /DIR: track 30.5 -> 33.7 mm
- net /MS1: track 27.2 -> 25.6 mm
- net +3V3: track 23.2 -> 24.8 mm
- net GND: track 39.9 -> 40.9 mm
- net /STEP: track 29.4 -> 28.4 mm
- net /INDEX: track 22.5 -> 23.5 mm
- net /PDN_UART: track 21.4 -> 22.3 mm
- net /MS2: track 26.2 -> 25.5 mm

Commit message: added lcsc field to components for ibom, also changed r5 to 33k
Parts:
- R2, R3: value R -> 0.75
- R5: value R -> 33k
Changed lines of the file:
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@@
     (descr "Capacitor SMD 0603 (1608 Metric), square (rectangular) end terminal, IPC_7351 nominal with elongated pad for handsoldering. (Body size source: IPC-SM-782 page 76, https://www.pcb-3d.com/wordpress/wp-content/uploads/ipc-sm-782a_amendment_1_and_2.pdf), generated with kicad-footprint-generator")
     (tags "capacitor handsolder")
+    (property "LCSC" "C1591")
     (property "Sheetfile" "tmc2208-breakout.kicad_sch")
     (property "Sheetname" "")
@@
     (descr "JST XH series connector, B4B-XH-A (http://www.jst-mfg.com/product/pdf/eng/eXH.pdf), generated with kicad-footprint-generator")
     (tags "connector JST XH vertical")
+    (property "LCSC" "C144395")
     (property "Sheetfile" "tmc2208-breakout.kicad_sch")
     (property "Sheetname" "")
@@
     (descr "Resistor SMD 0603 (1608 Metric), square (rectangular) end terminal, IPC_7351 nominal with elongated pad for handsoldering. (Body size source: IPC-SM-782 page 72, https://www.pcb-3d.com/wordpress/wp-content/uploads/ipc-sm-782a_amendment_1_and_2.pdf), generated with kicad-footprint-generator")
     (tags "resistor handsolder")
+    (property "LCSC" "C100044")
     (property "Sheetfile" "tmc2208-breakout.kicad_sch")
     (property "Sheetname" "")
@@
     (descr "Capacitor SMD 0603 (1608 Metric), square (rectangular) end terminal, IPC_7351 nominal with elongated pad for handsoldering. (Body size source: IPC-SM-782 page 76, https://www.pcb-3d.com/wordpress/wp-content/uploads/ipc-sm-782a_amendment_1_and_2.pdf), generated with kicad-footprint-generator")
     (tags "capacitor handsolder")
+    (property "LCSC" "C23630")
     (property "Sheetfile" "tmc2208-breakout.kicad_sch")
     (property "Sheetname" "")
@@
   (footprint "TMC2208-LA:TMC2208-LA" (layer "F.Cu")
     (at 157 61)
+    (property "LCSC" "C115944")
     (property "Sheetfile" "tmc2208-breakout.kicad_sch")
     (property "Sheetname" "")
@@
     (descr "Resistor SMD 0603 (1608 Metric), square (rectangular) end terminal, IPC_7351 nominal with elongated pad for handsoldering. (Body size source: IPC-SM-782 page 72, https://www.pcb-3d.com/wordpress/wp-content/uploads/ipc-sm-782a_amendment_1_and_2.pdf), generated with kicad-footprint-generator")
     (tags "resistor handsolder")
+    (property "LCSC" "C175689")
     (property "Sheetfile" "tmc2208-breakout.kicad_sch")
     (property "Sheetname" "")
@@
       (effects (font (size 1 1) (thickness 0.15)))
     )
-    (fp_text value "R" (at 0 1.43 90) (layer "F.Fab")
+    (fp_text value "0.75" (at 0 1.43 90) (layer "F.Fab")
       (effects (font (size 1 1) (thickness 0.15)))
     )
@@
     (descr "Resistor SMD 0603 (1608 Metric), square (rectangular) end terminal, IPC_7351 nominal with elongated pad for handsoldering. (Body size source: IPC-SM-782 page 72, https://www.pcb-3d.com/wordpress/wp-content/uploads/ipc-sm-782a_amendment_1_and_2.pdf), generated with kicad-footprint-generator")
     (tags "resistor handsolder")
+    (property "LCSC" "C100044")
     (property "Sheetfile" "tmc2208-breakout.kicad_sch")
     (property "Sheetname" "")
@@
     (descr "Capacitor SMD 0603 (1608 Metric), square (rectangular) end terminal, IPC_7351 nominal with elongated pad for handsoldering. (Body size source: IPC-SM-782 page 76, https://www.pcb-3d.com/wordpress/wp-content/uploads/ipc-sm-782a_amendment_1_and_2.pdf), generated with kicad-footprint-generator")
     (tags "capacitor handsolder")
+    (property "LCSC" "C1591")
     (property "Sheetfile" "tmc2208-breakout.kicad_sch")
     (property "Sheetname" "")
@@
     (descr "Through hole straight pin header, 1x11, 2.54mm pitch, single row")
     (tags "Through hole pin header THT 1x11 2.54mm single row")
+    (property "LCSC" "C429959")
     (property "Sheetfile" "tmc2208-breakout.kicad_sch")
     (property "Sheetname" "")
@@
     (descr "Resistor SMD 0603 (1608 Metric), square (rectangular) end terminal, IPC_7351 nominal with elongated pad for handsoldering. (Body size source: IPC-SM-782 page 72, https://www.pcb-3d.com/wordpress/wp-content/uploads/ipc-sm-782a_amendment_1_and_2.pdf), generated with kicad-footprint-generator")
     (tags "resistor handsolder")
+    (property "LCSC" "C175689")
     (property "Sheetfile" "tmc2208-breakout.kicad_sch")
     (property "Sheetname" "")
@@
       (effects (font (size 1 1) (thickness 0.15)))
     )
-    (fp_text value "R" (at 0 1.43 90) (layer "F.Fab")
+    (fp_text value "0.75" (at 0 1.43 90) (layer "F.Fab")
       (effects (font (size 1 1) (thickness 0.15)))
     )
@@
     (descr "Capacitor SMD 0603 (1608 Metric), square (rectangular) end terminal, IPC_7351 nominal with elongated pad for handsoldering. (Body size source: IPC-SM-782 page 76, https://www.pcb-3d.com/wordpress/wp-content/uploads/ipc-sm-782a_amendment_1_and_2.pdf), generated with kicad-footprint-generator")
     (tags "capacitor handsolder")
+    (property "LCSC" "C1591")
     (property "Sheetfile" "tmc2208-breakout.kicad_sch")
     (property "Sheetname" "")
@@
     (descr "Resistor SMD 0603 (1608 Metric), square (rectangular) end terminal, IPC_7351 nominal with elongated pad for handsoldering. (Body size source: IPC-SM-782 page 72, https://www.pcb-3d.com/wordpress/wp-content/uploads/ipc-sm-782a_amendment_1_and_2.pdf), generated with kicad-footprint-generator")
     (tags "resistor handsolder")
+    (property "LCSC" "C100044")
     (property "Sheetfile" "tmc2208-breakout.kicad_sch")
     (property "Sheetname" "")
@@
     (descr "Resistor SMD 0603 (1608 Metric), square (rectangular) end terminal, IPC_7351 nominal with elongated pad for handsoldering. (Body size source: IPC-SM-782 page 72, https://www.pcb-3d.com/wordpress/wp-content/uploads/ipc-sm-782a_amendment_1_and_2.pdf), generated with kicad-footprint-generator")
     (tags "resistor handsolder")
+    (property "LCSC" "C100044")
     (property "Sheetfile" "tmc2208-breakout.kicad_sch")
     (property "Sheetname" "")
@@
     (descr "Capacitor SMD 0603 (1608 Metric), square (rectangular) end terminal, IPC_7351 nominal with elongated pad for handsoldering. (Body size source: IPC-SM-782 page 76, https://www.pcb-3d.com/wordpress/wp-content/uploads/ipc-sm-782a_amendment_1_and_2.pdf), generated with kicad-footprint-generator")
     (tags "capacitor handsolder")
+    (property "LCSC" "C106222")
     (property "Sheetfile" "tmc2208-breakout.kicad_sch")
     (property "Sheetname" "")
@@
     (descr "Terminal Block Phoenix MKDS-1,5-2, 2 pins, pitch 5mm, size 10x9.8mm^2, drill diamater 1.3mm, pad diameter 2.6mm, see http://www.farnell.com/datasheets/100425.pdf, script-generated using https://github.com/pointhi/kicad-footprint-generator/scripts/TerminalBlock_Phoenix")
     (tags "THT Terminal Block Phoenix MKDS-1,5-2 pitch 5mm size 10x9.8mm^2 drill 1.3mm pad 2.6mm")
+    (property "LCSC" "C8404")
     (property "Sheetfile" "tmc2208-breakout.kicad_sch")
     (property "Sheetname" "")
@@
     (descr "SMD capacitor, aluminum electrolytic, Panasonic C55, 6.3x5.4mm")
     (tags "capacitor electrolytic")
+    (property "LCSC" "C129250")
     (property "Sheetfile" "tmc2208-breakout.kicad_sch")
     (property "Sheetname" "")
@@
     (descr "Capacitor SMD 0603 (1608 Metric), square (rectangular) end terminal, IPC_7351 nominal with elongated pad for handsoldering. (Body size source: IPC-SM-782 page 76, https://www.pcb-3d.com/wordpress/wp-content/uploads/ipc-sm-782a_amendment_1_and_2.pdf), generated with kicad-footprint-generator")
     (tags "capacitor handsolder")
+    (property "LCSC" "C1591")
     (property "Sheetfile" "tmc2208-breakout.kicad_sch")
     (property "Sheetname" "")
@@
     (descr "Resistor SMD 0603 (1608 Metric), square (rectangular) end terminal, IPC_7351 nominal with elongated pad for handsoldering. (Body size source: IPC-SM-782 page 72, https://www.pcb-3d.com/wordpress/wp-content/uploads/ipc-sm-782a_amendment_1_and_2.pdf), generated with kicad-footprint-generator")
     (tags "resistor handsolder")
+    (property "LCSC" "C25593")
     (property "Sheetfile" "tmc2208-breakout.kicad_sch")
     (property "Sheetname" "")
@@
       (effects (font (size 1 1) (thickness 0.15)))
     )
-    (fp_text value "R" (at 0 1.43) (layer "F.Fab")
+    (fp_text value "33k" (at 0 1.43) (layer "F.Fab")
       (effects (font (size 1 1) (thickness 0.15)))
     )
@@
     (descr "Resistor SMD 0603 (1608 Metric), square (rectangular) end terminal, IPC_7351 nominal with elongated pad for handsoldering. (Body size source: IPC-SM-782 page 72, https://www.pcb-3d.com/wordpress/wp-content/uploads/ipc-sm-782a_amendment_1_and_2.pdf), generated with kicad-footprint-generator")
     (tags "resistor handsolder")
-    (property "Sheetfile" "tmc2208-breakout.kicad_sch")
-    (property "Sheetname" "")
+    (property "LCSC" "C100044")
+    (property "Sheetfile" "tmc2208-breakout.kicad_sch")
+    (property "Sheetname" "")
